Commit message: Refactor robot configuration to use origin_xyz and origin_rpy for positioning in launch file and URDF

File: src/dual_ur_simulation/urdf/ur.urdf.xacro (robot description, xacro)
@@ -15,4 +15,6 @@
    <xacro:arg name="simulation_controllers" default="" />
    <xacro:arg name="ros_namespace" default="" />
+   <xacro:arg name="origin_xyz" default="0 0 0"/>
+   <xacro:arg name="origin_rpy" default="0 0 0"/>
    <!-- UR Macro einbinden -->
    <xacro:include filename="$(find ur_description)/urdf/ur_macro.xacro"/>
@@ -34,5 +36,5 @@
      safety_k_position="$(arg safety_k_position)"
      force_abs_paths="true">
-     <origin xyz="0 0 0" rpy="0 0 0" />
+     <origin xyz="$(arg origin_xyz)" rpy="$(arg origin_rpy)" />
    </xacro:ur_robot>
    <!-- Gazebo Plugin -->

Commit message: Update Dockerfile and URDF to integrate ros2_control and Robotiq gripper support

File: src/dual_ur_simulation/urdf/ur.urdf.xacro (robot description, xacro)
@@ -19,4 +19,6 @@
    <!-- UR Macro einbinden -->
    <xacro:include filename="$(find ur_description)/urdf/ur_macro.xacro"/>
+   <xacro:include filename="$(find robotiq_description)/urdf/ur_to_robotiq_adapter.urdf.xacro" />
+   <xacro:include filename="$(find robotiq_description)/urdf/robotiq_2f_85_macro.urdf.xacro" />
    <!-- ros2_control einbinden -->
    <xacro:include filename="$(find dual_ur_simulation)/urdf/ur_ros2_control.xacro"/>
@@ -38,4 +40,16 @@
      <origin xyz="$(arg origin_xyz)" rpy="$(arg origin_rpy)" />
    </xacro:ur_robot>
+   <xacro:ur_to_robotiq
+     prefix="$(arg tf_prefix)"
+     connected_to="$(arg tf_prefix)tool0"/>
+   <xacro:robotiq_gripper
+     name="$(arg tf_prefix)RobotiqGripperHardwareInterface"
+     prefix="$(arg tf_prefix)"
+     parent="$(arg tf_prefix)gripper_mount_link"
+     use_fake_hardware="false"
+     sim_gazebo="true"
+     include_ros2_control="false">
+     <origin xyz="0 0 0" rpy="0 0 0"/>
+   </xacro:robotiq_gripper>
    <!-- Gazebo Plugin -->
    <gazebo reference="world">
